File: X16-ESC-Adapter.sch (EAGLE design)
At the start: 9 parts, among them J1 BM08B-SRSS-TB(LF)(SN)

Commit message: Minh Update 1
Parts:
- renumbered 600 to R1, HOPE to 12V_LED
Connections:
- net GND: now also J1.SHIELD
Changed lines of the file:
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@@
 <layers>
 <layer number="1" name="Top" color="4" fill="1" visible="no" active="no"/>
+<layer number="2" name="Route2" color="1" fill="3" visible="no" active="no"/>
+<layer number="3" name="Route3" color="4" fill="3" visible="no" active="no"/>
+<layer number="4" name="Route4" color="1" fill="4" visible="no" active="no"/>
+<layer number="5" name="Route5" color="4" fill="4" visible="no" active="no"/>
+<layer number="6" name="Route6" color="1" fill="8" visible="no" active="no"/>
+<layer number="7" name="Route7" color="4" fill="8" visible="no" active="no"/>
+<layer number="8" name="Route8" color="1" fill="2" visible="no" active="no"/>
+<layer number="9" name="Route9" color="4" fill="2" visible="no" active="no"/>
+<layer number="10" name="Route10" color="1" fill="7" visible="no" active="no"/>
+<layer number="11" name="Route11" color="4" fill="7" visible="no" active="no"/>
+<layer number="12" name="Route12" color="1" fill="5" visible="no" active="no"/>
+<layer number="13" name="Route13" color="4" fill="5" visible="no" active="no"/>
+<layer number="14" name="Route14" color="1" fill="6" visible="no" active="no"/>
+<layer number="15" name="Route15" color="4" fill="6" visible="no" active="no"/>
 <layer number="16" name="Bottom" color="1" fill="1" visible="no" active="no"/>
 <layer number="17" name="Pads" color="2" fill="1" visible="no" active="no"/>
@@
 <part name="ESC3" library="X16-ESC-Adapter" deviceset="CONN_1824750000" device=""/>
 <part name="ESC4" library="X16-ESC-Adapter" deviceset="CONN_1824750000" device=""/>
-<part name="600" library="SparkFun-Resistors" library_urn="urn:adsk.eagle:library:532" deviceset="0.1OHM" device="-0603-1/3W-1%" package3d_urn="urn:adsk.eagle:package:41389018/1" value="600"/>
-<part name="HOPE" library="led" library_urn="urn:adsk.eagle:library:259" deviceset="LED" device="CHIPLED_0805" package3d_urn="urn:adsk.eagle:package:15821/2"/>
+<part name="R1" library="SparkFun-Resistors" library_urn="urn:adsk.eagle:library:532" deviceset="0.1OHM" device="-0603-1/3W-1%" package3d_urn="urn:adsk.eagle:package:41389018/1" value="600"/>
+<part name="12V_LED" library="led" library_urn="urn:adsk.eagle:library:259" deviceset="LED" device="CHIPLED_0805" package3d_urn="urn:adsk.eagle:package:15821/2"/>
 <part name="J1" library="X16-ESC-Adapter" deviceset="BM08B-SRSS-TB(LF)(SN)" device=""/>
 </parts>
@@
 <attribute name="LAST_DATE_TIME" x="44.45" y="-82.55" size="2.286" layer="94" font="vector"/>
 <attribute name="SHEET" x="58.42" y="-87.63" size="2.54" layer="94" font="vector"/>
-<attribute name="DESIGNER" x="89.1" y="-82.55" size="2.54" layer="94" font="vector"/>
 </instance>
 <instance part="ESC1" gate="A" x="-66.04" y="27.94" smashed="yes">
@@
 <attribute name="NAME" x="-39.7256" y="9.9314" size="2.0828" layer="95" ratio="6" rot="SR180"/>
 </instance>
-<instance part="600" gate="G$1" x="-55.88" y="53.34" smashed="yes">
+<instance part="R1" gate="G$1" x="-55.88" y="53.34" smashed="yes">
 <attribute name="NAME" x="-55.88" y="54.864" size="1.778" layer="95" font="vector" align="bottom-center"/>
 <attribute name="VALUE" x="-55.88" y="51.816" size="1.778" layer="96" font="vector" align="top-center"/>
 </instance>
-<instance part="HOPE" gate="G$1" x="-45.72" y="53.34" smashed="yes" rot="R90">
+<instance part="12V_LED" gate="G$1" x="-45.72" y="53.34" smashed="yes" rot="R90">
 <attribute name="NAME" x="-41.148" y="56.896" size="1.778" layer="95" rot="R180"/>
 <attribute name="VALUE" x="-41.148" y="59.055" size="1.778" layer="96" rot="R180"/>
@@
 </segment>
 <segment>
-<pinref part="600" gate="G$1" pin="1"/>
+<pinref part="R1" gate="G$1" pin="1"/>
 <wire x1="-60.96" y1="53.34" x2="-63.5" y2="53.34" width="0.1524" layer="91"/>
 <label x="-63.5" y="53.34" size="1.778" layer="95" rot="R180" xref="yes"/>
@@
 <wire x1="-40.64" y1="53.34" x2="-38.1" y2="53.34" width="0.1524" layer="91"/>
 <label x="-38.1" y="53.34" size="1.778" layer="95" xref="yes"/>
-<pinref part="HOPE" gate="G$1" pin="C"/>
+<pinref part="12V_LED" gate="G$1" pin="C"/>
 </segment>
 <segment>
@@
 <wire x1="-40.64" y1="-53.34" x2="-38.1" y2="-53.34" width="0.1524" layer="91"/>
 <label x="-38.1" y="-53.34" size="1.778" layer="95" xref="yes"/>
+</segment>
+<segment>
+<wire x1="-40.64" y1="-33.02" x2="-38.1" y2="-33.02" width="0.1524" layer="91"/>
+<label x="-38.1" y="-33.02" size="1.778" layer="95" xref="yes"/>
+<pinref part="J1" gate="G$1" pin="SHIELD"/>
 </segment>
 </net>
@@
 <net name="N$1" class="0">
 <segment>
-<pinref part="600" gate="G$1" pin="2"/>
+<pinref part="R1" gate="G$1" pin="2"/>
 <wire x1="-50.8" y1="53.34" x2="-48.26" y2="53.34" width="0.1524" layer="91"/>
-<pinref part="HOPE" gate="G$1" pin="A"/>
-</segment>
-</net>
+<pinref part="12V_LED" gate="G$1" pin="A"/>
+</segment>
+</net>

Commit message: Create GERBER files
Parts:
- R1: value 600 -> 0.1
Changed lines of the file:
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@@
 <part name="ESC3" library="X16-ESC-Adapter" deviceset="CONN_1824750000" device=""/>
 <part name="ESC4" library="X16-ESC-Adapter" deviceset="CONN_1824750000" device=""/>
-<part name="R1" library="SparkFun-Resistors" library_urn="urn:adsk.eagle:library:532" deviceset="0.1OHM" device="-0603-1/3W-1%" package3d_urn="urn:adsk.eagle:package:41389018/1" value="600"/>
+<part name="R1" library="SparkFun-Resistors" library_urn="urn:adsk.eagle:library:532" deviceset="0.1OHM" device="-0603-1/3W-1%" package3d_urn="urn:adsk.eagle:package:41389018/1" value="0.1"/>
 <part name="12V_LED" library="led" library_urn="urn:adsk.eagle:library:259" deviceset="LED" device="CHIPLED_0805" package3d_urn="urn:adsk.eagle:package:15821/2"/>
 <part name="J1" library="X16-ESC-Adapter" deviceset="BM08B-SRSS-TB(LF)(SN)" device=""/>
